File: LEDModule.kicad_pcb (KiCad board)
At the start: 2 copper layers, 29 x 32.2 mm, 12 parts, among them J1 Conn_01x02, Q1 BC847BS

Commit message: Updated package size of R1. Added LCSC BOM.
Parts:
- R1: footprint Resistor_SMD:R_0201_0603Metric -> Resistor_SMD:R_0603_1608Metric
- moved R1 0.50 mm to (79.5, 92.2)
Routing:
- net Net-(Q1-Pad5): track 5.01 -> 4.01 mm
Other:
- board text added: "LED Module 11-14V DC 20mA v0.1 2023-01-05"
- board text removed: "LED Module 11-14V DC 20mA v0.0 2022-12-18"
